Commit message: RTABMap code

File: urdf/_d435.gazebo.xacro (robot description, xacro)
@@ -27,6 +27,6 @@
           <horizontal_fov>${69.4*deg_to_rad}</horizontal_fov>
           <image>
-            <width>1280</width>
-            <height>720</height>
+            <width>1920</width>
+            <height>1080</height>
             <format>RGB_INT8</format>
           </image>
@@ -49,5 +49,5 @@
           <horizontal_fov>${85.2*deg_to_rad}</horizontal_fov>
           <image>
-            <width>1080</width>
+            <width>1280</width>
             <height>720</height>
             <format>L_INT8</format>
@@ -93,6 +93,6 @@
           <horizontal_fov>${69.4*deg_to_rad}</horizontal_fov>
           <image>
-            <width>1080</width>
-            <height>720</height>
+            <width>1920</width>
+            <height>1080</height>
           </image>
           <clip>
@@ -130,9 +130,8 @@
       	<infrared2OpticalframeName>${infrared2_optical_frame}</infrared2OpticalframeName>
       	<rangeMinDepth>0.2</rangeMinDepth>
-      	<rangeMaxDepth>3.0</rangeMaxDepth>
+      	<rangeMaxDepth>10.0</rangeMaxDepth>
       	<pointCloud>true</pointCloud>
       	<pointCloudTopicName>depth/points</pointCloudTopicName>
-      	<pointCloudCutoff>0.2</pointCloudCutoff>
-        <pointCloudCutoffMax>3</pointCloudCutoffMax>
+      	<pointCloudCutoff>0.5</pointCloudCutoff>
       </plugin>
     </gazebo>

File: urdf/m6.urdf.xacro (robot description, xacro)
@@ -170,5 +170,5 @@
       <geometry>
         <mesh
-          filename="package://xMonsterCPG/meshes/camera_mount.STL" scale="1 1 1"/>
+          filename="package://xMonsterCPG/meshes/camera_mount.STL" scale="2 2 2"/>
       </geometry>
       <material
@@ -184,5 +184,5 @@
       <geometry>
         <mesh
-          filename="package://xMonsterCPG/meshes/camera_mount.STL" scale="1 1 1"/>
+          filename="package://xMonsterCPG/meshes/camera_mount.STL" scale="2 2 2"/>
       </geometry>
     </collision>
@@ -226,5 +226,5 @@
     <!-- Create camera instance 0.05 0.0 0.715" rpy="0 0.9 0" -->
     <xacro:sensor_d435 parent="base_link">
-        <origin xyz="0.1 0.0 0.3" rpy="0 0.3 0" />
+        <origin xyz="0.15 0.0 0.48" rpy="0 0 0" />
     </xacro:sensor_d435>
     <gazebo>
